Commit message: first edit changing disc as joint

File: src/primo-arm-r01/urdf/output.urdf (robot description, URDF)
Before this commit: robot primio_arm_r01, 12 links, 11 joints
Links:
- link disc_9: geometry visual cylinder length=0.005 radius=0.011
- link link_10: geometry visual box size=0.02 0.02 0.19; visual cylinder length=0.005 radius=0.011
- link link_11: geometry visual box size=0.02 0.02 0.15; visual cylinder length=0.005 radius=0.011
- link link_12: geometry visual box size=0.02 0.02 0.11; visual cylinder length=0.005 radius=0.011
- link link_13: geometry visual box size=0.02 0.02 0.0; visual cylinder length=0.005 radius=0.011
- link motor_block10: geometry visual box size=0.032 0.032 0.05
- link motor_block11: geometry visual box size=0.032 0.032 0.05; visual cylinder length=0.005 radius=0.011
- link motor_block12: geometry visual box size=0.032 0.032 0.05; visual cylinder length=0.005 radius=0.011
- link motor_block13: geometry visual box size=0.032 0.032 0.05
- link motor_block9: geometry visual box size=0.032 0.032 0.05
Joints:
- joint disc9_to_motor_block10: origin xyz=0 0 ${disc_thickness/2} rpy=0 0 0 -> xyz=0 0 0.0025 rpy=0 0 0
- joint joint_10: origin xyz=${motor_offset + link_side/2 + disc_thickness} 0 ${motor_height - 0.020} rpy=0 0 0 -> xyz=0.031000000000000003 0 0.030000000000000002 rpy=0 0 0
- joint joint_10_5: origin xyz=0 0 ${link1_length} rpy=3.14159 3.14159 0 -> xyz=0 0 0.19 rpy=3.14159 3.14159 0
- joint joint_11: origin xyz=${motor_offset + link_side/2 + disc_thickness} 0 ${motor_height + disc_thickness - 0.020} rpy=0 0 0 -> xyz=0.031000000000000003 0 0.035 rpy=0 0 0
- joint joint_11_5: origin xyz=0 0 ${link2_length} rpy=3.14159 3.14159 0 -> xyz=0 0 0.15 rpy=3.14159 3.14159 0
- joint joint_12: origin xyz=${motor_offset + link_side/2 + disc_thickness} 0 ${motor_height + disc_thickness - 0.020} rpy=0 0 0 -> xyz=0.031000000000000003 0 0.035 rpy=0 0 0
- joint joint_12_5: origin xyz=0 0 ${link3_length} rpy=3.14159 3.14159 0 -> xyz=0 0 0.11 rpy=3.14159 3.14159 0
- joint joint_13: origin xyz=${link_side/2} 0 ${motor_size + disc_thickness} rpy=0 0 0 -> xyz=0.01 0 0.037 rpy=0 0 0
- joint joint_9: origin xyz=${link_side/2} 0 ${motor_size + disc_thickness/2} rpy=0 0 0 -> xyz=0.01 0 0.0345 rpy=0 0 0
